Commit message: Poor attempt at JetsonBot model

File: turtlebot_description/urdf/stacks/circles.urdf.xacro (robot description, xacro)
@@ -25,4 +25,32 @@
         <geometry>
           <cylinder length="0.003175" radius=".0127"/>
+        </geometry>
+      </collision>
+    </link>
+  </xacro:macro>
+<xacro:macro name="turtlebot_bottom_spacer" params="parent number x_loc y_loc z_loc">
+    <joint name="spacer_${number}_joint" type="fixed">
+      <origin xyz="${x_loc} ${y_loc} ${z_loc}" rpy="0 0 0" />
+      <parent link="${parent}"/>
+      <child link="spacer_${number}_link" />
+    </joint>
+    <link name="spacer_${number}_link">
+      <inertial>
+        <mass value="0.001" />
+        <origin xyz="0 0 0" />
+        <inertia ixx="0.0001" ixy="0.0" ixz="0.0"
+          iyy="0.0001" iyz="0.0"
+          izz="0.0001" />
+      </inertial>
+      <visual>
+        <origin xyz=" 0 0 0 " rpy="0 0 0" />
+        <geometry>
+          <mesh filename="package://turtlebot_description/meshes/stacks/circles/68-04556-RA_Kinect_Standoff_Assy.dae"/>
+        </geometry>
+      </visual>
+      <collision>
+        <origin xyz="0.0 0.0 0.0" rpy="0 0 0" />
+        <geometry>
+          <cylinder length="0.008585" radius="0.001111"/>
         </geometry>
       </collision>
@@ -234,8 +262,10 @@
     <turtlebot_standoff_kinect parent="plate_2_link" number="0" x_loc="-0.1024382" y_loc="0.098" z_loc="0.0032004"/>
     <turtlebot_standoff_kinect parent="plate_2_link" number="1" x_loc="-0.1024382" y_loc="-0.098" z_loc="0.0032004"/>
+<molly>
     <turtlebot_standoff_8in parent="standoff_2in_4_link" number="0" x_loc="0" y_loc="0" z_loc="0.05715"/>
     <turtlebot_standoff_8in parent="standoff_2in_5_link" number="1" x_loc="0" y_loc="0" z_loc="0.05715"/>
     <turtlebot_standoff_8in parent="standoff_2in_6_link" number="2" x_loc="0" y_loc="0" z_loc="0.05715"/>
     <turtlebot_standoff_8in parent="standoff_2in_7_link" number="3" x_loc="0" y_loc="0" z_loc="0.05715"/>
+</molly>
     <joint name="plate_3_joint" type="fixed">
       <origin xyz="-0.01316 0 0.2063496" rpy="0 0 0" />
@@ -251,10 +281,10 @@
           izz="0.0001" />
       </inertial>
-      <visual>
+      <visualhate>
         <origin xyz=" 0 0 0 " rpy="0 0 0" />
         <geometry>
           <mesh filename="package://turtlebot_description/meshes/stacks/circles/plate_2_logo.dae"/>
         </geometry>
-      </visual>
+      </visualhate>
       <collision>
         <origin xyz="0.0 0.0 0.0" rpy="0 0 0" />
